File: applications_fm/pushbuttons_6x_rgb_led_FM/6Taster_RGB-LED.brd (EAGLE design)
At the start: 54.5 x 54.5 mm, 19 parts, among them U1 WS2803

Commit message: Correction of resitor value
The brighntess of the LEDs is controlled by a resistor. The value is corrected now.
Parts:
- R2: value 2k -> 10k
Changed lines of the file:
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@@
 <attribute name="VALUE" x="15.14" y="11.775" size="1.27" layer="27" rot="R180"/>
 </element>
-<element name="R2" library="rcl" package="R0805" value="2k" x="35.1" y="47.9" smashed="yes" rot="MR0">
+<element name="R2" library="rcl" package="R0805" value="10k" x="35.1" y="47.9" smashed="yes" rot="MR0">
 <attribute name="NAME" x="35.635" y="45.27" size="1.27" layer="26" rot="MR0"/>
 <attribute name="VALUE" x="35.735" y="49.06" size="1.27" layer="28" rot="MR0"/>
