File: modules_lpc1115_fm/io-16x-fused-fm/io-16x-fused-fm.brd (EAGLE design)
At the start: 46.8 x 48.9 mm, 143 parts, among them IC5 LPC1115, IC6 ATAES132A-SHEQ-T, J1 62000611622, J2 1771017, J3 1770953, Q3 ASFL, U3 EEPROM, X1 MICROMATCH-10SMD

Commit message: [IO16xFM] - made .sch nicer to read
Connections:
- net +3V3: now also J3.3, J3.4; no longer J3.1, J3.2
- net GND: now also J3.1, J3.2; no longer J3.3, J3.4
Routing:
- net IO6: track 23.7 -> 20.1 mm
- net +3V3: track 289.4 -> 287.0 mm
Other:
- board text added: "www.selfbus.org IO module 16x fused v1.0.0"
- board text removed: "www.selfbus.org IO module 16x fused beta"
Changed lines of the file:
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@@
 IO module
 16x fused
-beta</text>
+v1.0.0</text>
 <text x="4.7" y="7" size="1.016" layer="51">GND
 3V3</text>
@@
 <contactref element="JP23" pad="2"/>
 <contactref element="JP22" pad="4"/>
-<contactref element="J3" pad="3"/>
-<contactref element="J3" pad="4"/>
 <contactref element="X1" pad="1"/>
 <contactref element="D5" pad="A"/>
@@
 <via x="32.6" y="25.8" extent="1-16" drill="0.35"/>
 <via x="11.7" y="21.6" extent="1-16" drill="0.35"/>
-<wire x1="4.5" y1="15.6" x2="1.4" y2="15.6" width="0.4064" layer="16"/>
 <via x="5" y="5.5" extent="1-16" drill="0.35"/>
 <via x="8.4" y="4" extent="1-16" drill="0.35"/>
@@
 <via x="27.8" y="45.7" extent="1-16" drill="0.35"/>
 <via x="30.6" y="23.6" extent="1-16" drill="0.35"/>
+<contactref element="J3" pad="2"/>
+<contactref element="J3" pad="1"/>
+<wire x1="1.4" y1="13.1" x2="4.5" y2="13.1" width="0.4064" layer="16"/>
 </signal>
 <signal name="EIB_OUT">
@@
 <contactref element="IC5" pad="13"/>
 <contactref element="R73" pad="2"/>
-<wire x1="25.0508" y1="12.1" x2="22.1" y2="15.0508" width="0.2" layer="1"/>
-<wire x1="22.1" y1="15.0508" x2="22.1" y2="17.6" width="0.2" layer="1"/>
-<via x="22.1" y="17.6" extent="1-16" drill="0.35"/>
-<wire x1="22.1" y1="17.6" x2="24.1" y2="17.6" width="0.2" layer="16"/>
-<wire x1="29.5" y1="23" x2="24.1" y2="17.6" width="0.2" layer="16"/>
+<wire x1="25.5" y1="18.5" x2="25.5" y2="12.5492" width="0.2" layer="1"/>
+<wire x1="25.0508" y1="12.1" x2="25.5" y2="12.5492" width="0.2" layer="1"/>
+<via x="25.5" y="18.5" extent="1-16" drill="0.35"/>
+<wire x1="25.5" y1="18.5" x2="25.5" y2="19" width="0.2" layer="16"/>
+<wire x1="29.5" y1="23" x2="25.5" y2="19" width="0.2" layer="16"/>
 <wire x1="29.7" y1="27.4" x2="29.5" y2="27.2" width="0.2" layer="16"/>
 <wire x1="29.5" y1="27.2" x2="29.5" y2="23" width="0.2" layer="16"/>
@@
 <contactref element="JP22" pad="3"/>
 <contactref element="LED6" pad="A"/>
-<contactref element="J3" pad="2"/>
-<contactref element="J3" pad="1"/>
 <wire x1="30.75" y1="29.8" x2="30.75" y2="31.9" width="0.254" layer="1"/>
 <contactref element="X1" pad="2"/>
@@
 <wire x1="20.0306" y1="34.0197875" x2="19.5797875" y2="34.4706" width="0.3048" layer="1"/>
 <wire x1="19.5797875" y1="34.4706" x2="18.18506875" y2="34.4706" width="0.3048" layer="1"/>
-<wire x1="1.1428" y1="13.1" x2="1.1428" y2="10.382225" width="0.4064" layer="1"/>
 <wire x1="20.837575" y1="2.3198" x2="21.831" y2="3.313225" width="0.4064" layer="1"/>
 <wire x1="21.831" y1="3.313225" x2="21.831" y2="5.481" width="0.4064" layer="1"/>
 <wire x1="22.9" y1="6.55" x2="21.831" y2="5.481" width="0.4064" layer="1"/>
-<wire x1="1.1428" y1="10.382225" x2="9.205225" y2="2.3198" width="0.4064" layer="1"/>
+<wire x1="6.9125125" y1="4.6125125" x2="9.205225" y2="2.3198" width="0.4064" layer="1"/>
 <wire x1="9.205225" y1="2.3198" x2="20.837575" y2="2.3198" width="0.4064" layer="1"/>
 <wire x1="31.65" y1="13.4" x2="32.063025" y2="13.4" width="0.4064" layer="1"/>
@@
 <wire x1="31.24353125" y1="40.3938" x2="28.4538" y2="40.3938" width="0.4064" layer="16"/>
 <wire x1="28.4538" y1="40.3938" x2="26.76" y2="38.7" width="0.4064" layer="16"/>
-<wire x1="1.4" y1="13.1" x2="4.5" y2="13.1" width="0.4064" layer="16"/>
-<wire x1="4.5" y1="13.1" x2="1.1428" y2="13.1" width="0.4064" layer="1"/>
 <wire x1="22.9" y1="7.1" x2="24.1" y2="8.3" width="0.4064" layer="1"/>
 <wire x1="22.9" y1="6.55" x2="22.9" y2="7.1" width="0.4064" layer="1"/>
@@
 <wire x1="30.3302" y1="48.0802" x2="29.55" y2="47.3" width="0.4064" layer="1"/>
 <wire x1="29.55" y1="46.7" x2="29.55" y2="47.3" width="0.4064" layer="1"/>
-<wire x1="37.35" y1="46.8" x2="38.125" y2="46.025" width="0.4064" layer="1"/>
+<wire x1="37.35" y1="46.8" x2="37.3794" y2="46.7706" width="0.4064" layer="1"/>
 <wire x1="37.35" y1="46.8" x2="35.65" y2="46.8" width="0.4064" layer="1"/>
 <wire x1="40.85" y1="43.7001" x2="40.85" y2="42.8" width="0.4064" layer="1"/>
@@
 <wire x1="22.9" y1="6.4" x2="22.9" y2="6.55" width="0.254" layer="1"/>
 <wire x1="23.746" y1="5.554" x2="22.9" y2="6.4" width="0.254" layer="1"/>
-<wire x1="38.125" y1="46.025" x2="38.702253125" y2="46.025" width="0.4064" layer="1"/>
-<wire x1="38.702253125" y1="46.025" x2="40.12416875" y2="44.903828125" width="0.4064" layer="1"/>
-<wire x1="40.12416875" y1="44.903828125" x2="40.85" y2="44.177996875" width="0.4064" layer="1"/>
-<wire x1="40.85" y1="44.177996875" x2="40.85" y2="43.7001" width="0.4064" layer="1"/>
+<wire x1="37.3794" y1="46.7706" x2="40.85" y2="44.034053125" width="0.4064" layer="1"/>
+<wire x1="40.85" y1="44.034053125" x2="40.85" y2="43.7001" width="0.4064" layer="1"/>
+<contactref element="J3" pad="3"/>
+<contactref element="J3" pad="4"/>
+<wire x1="4.5" y1="15.6" x2="1.4" y2="15.6" width="0.4064" layer="16"/>
+<wire x1="6.4498" y1="13.777175" x2="4.626975" y2="15.6" width="0.4064" layer="1"/>
+<wire x1="4.5" y1="15.6" x2="4.626975" y2="15.6" width="0.4064" layer="1"/>
+<wire x1="6.4498" y1="5.075225" x2="6.9125125" y2="4.6125125" width="0.4064" layer="1"/>
+<wire x1="6.4498" y1="13.777175" x2="6.4498" y2="5.075225" width="0.4064" layer="1"/>
 </signal>
 <signal name="N$26">
@@
 <contactref element="J2" pad="13"/>
 <contactref element="J2" pad="14"/>
-<wire x1="6.415" y1="18.785" x2="6.415" y2="10.966" width="0.254" layer="1"/>
+<wire x1="6.415" y1="18.785" x2="6.415" y2="15.6" width="0.254" layer="1"/>
 <wire x1="4.5" y1="20.7" x2="6.415" y2="18.785" width="0.254" layer="1"/>
-<wire x1="6.415" y1="10.966" x2="7.69433125" y2="9.68666875" width="0.254" layer="1"/>
-<wire x1="8.326" y1="9.6867" x2="7.69433125" y2="9.68666875" width="0.254" layer="1"/>
+<wire x1="7.894321875" y1="9.686678125" x2="8.326" y2="9.6867" width="0.254" layer="1"/>
 <wire x1="4.5" y1="20.7" x2="1.4" y2="20.7" width="0.4064" layer="16"/>
+<wire x1="6.415" y1="15.6" x2="7.372" y2="14.643" width="0.254" layer="1"/>
+<wire x1="7.372" y1="14.643" x2="7.372" y2="14.4114875" width="0.254" layer="1"/>
+<wire x1="7.372" y1="14.4114875" x2="7.388" y2="14.3954875" width="0.254" layer="1"/>
+<wire x1="7.388" y1="14.3954875" x2="7.388" y2="10.193" width="0.254" layer="1"/>
+<wire x1="7.388" y1="10.193" x2="7.894321875" y2="9.686678125" width="0.254" layer="1"/>
 </signal>
 <signal name="IN6">
@@
 <contactref element="J2" pad="15"/>
 <contactref element="J2" pad="16"/>
-<wire x1="5.934" y1="16.766" x2="5.934" y2="9.966" width="0.254" layer="1"/>
+<wire x1="5.934" y1="16.766" x2="5.934" y2="15.2" width="0.254" layer="1"/>
 <wire x1="4.5" y1="18.2" x2="5.934" y2="16.766" width="0.254" layer="1"/>
-<wire x1="5.934" y1="9.966" x2="7.90666875" y2="7.99333125" width="0.254" layer="1"/>
 <wire x1="7.90666875" y1="7.99333125" x2="8.326" y2="7.9933" width="0.254" layer="1"/>
 <wire x1="1.4" y1="18.2" x2="4.5" y2="18.2" width="0.4064" layer="16"/>
+<wire x1="5.934" y1="15.2" x2="7.007" y2="14.127" width="0.254" layer="1"/>
+<wire x1="7.007" y1="14.127" x2="7.007" y2="8.893" width="0.254" layer="1"/>
+<wire x1="7.007" y1="8.893" x2="7.90666875" y2="7.99333125" width="0.254" layer="1"/>
 </signal>
 <signal name="IO4">
@@
 <wire x1="33.9" y1="19.4" x2="32.85" y2="18.35" width="0.2" layer="16"/>
 <wire x1="32.85" y1="18.35" x2="32.85" y2="18.15" width="0.2" layer="16"/>
-<wire x1="33.25" y1="21.2" x2="33.25" y2="20" width="0.2" layer="1"/>
-<wire x1="33.35" y1="19.9" x2="33.25" y2="20" width="0.2" layer="1"/>
-<wire x1="33.35" y1="19.9" x2="33.35" y2="18.7" width="0.2" layer="1"/>
-<wire x1="33.35" y1="18.7" x2="32.85" y2="18.2" width="0.2" layer="1"/>
+<wire x1="33.25" y1="21.2" x2="33.25" y2="18.6" width="0.2" layer="1"/>
+<wire x1="33.25" y1="18.6" x2="32.85" y2="18.2" width="0.2" layer="1"/>
 <wire x1="32.85" y1="18.2" x2="32.85" y2="18.15" width="0.2" layer="1"/>
 <via x="32.85" y="18.15" extent="1-16" drill="0.35"/>
