File: modules_lpc1115_fm/io-16x-fused-fm/io-16x-fused-fm.sch (EAGLE design)
At the start: 143 parts, among them IC5 LPC1115, IC6 ATAES132A-SHEQ-T, J1 62000611622, J2 1771017, J3 1770953, Q3 ASFL, U3 EEPROM, X1 MICROMATCH-10SMD

Commit message: [IO16xFM] - made .sch nicer to read
Connections:
- net +3V3: now also J3.2.1, J3.2.2; no longer J3.1.1, J3.1.2
- net GND: now also J3.1.1, J3.1.2; no longer J3.2.1, J3.2.2
Other:
- note added: "BOTTOM IOs"
- note added: "I2C - pullups already integrated"
- note added: "ISP interface"
- note added: "MCU with decoupling MLCCs and Oscillator"
- note added: "Pins for stabilization and heat dissipation of KNX breakout board"
- note added: "SPI"
- note added: "TOP IOs"
- note added: "connection to KNX breakout board"
- note added: "prog button and prog LED"
- note added: "v1.0"
- note removed: "Pins for stabilization and heat dissipation"
- moved on the sheet: C1, C2, C25, C26, C27, C28, C29, C30, C31, C32, C33, C34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
