File: applications_din/in_8x_24V_DC_2MU/2te8LED/2te8LED_v04.brd (EAGLE design)
At the start: 30.6 x 40.6 mm, 19 parts, among them IC1 74HC595D

Commit message: 3D models added
Parts:
- JP1: device pinhead:1X07 -> con-lsta:FE07
Changed lines of the file:
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@@
 <attribute name="NAME" x="17.533" y="2.4723" size="1.27" layer="26" ratio="10" rot="MR180"/>
 </element>
-<element name="IC1" library="74xx-eu" package="SO16" value="74HC595D" x="12.0385" y="17.7438" smashed="yes" rot="MR270">
+<element name="IC1" library="74xx-eu" library_urn="urn:adsk.eagle:library:85" package="SO16" package3d_urn="urn:adsk.eagle:package:2010/1" override_package3d_urn="urn:adsk.eagle:package:48524435/2" override_package_urn="urn:adsk.eagle:footprint:1637/1" value="74HC595D" x="12.0385" y="17.7438" smashed="yes" rot="MR270">
 <attribute name="NAME" x="10.3392" y="12.1021" size="1.27" layer="26" ratio="10" rot="MR180"/>
+<attribute name="POPULARITY" value="21" x="12.0385" y="17.7438" size="1.778" layer="28" rot="MR270" display="off"/>
 <attribute name="VALUE" x="12.7801" y="13.123" size="1.27" layer="27" ratio="10" rot="R90"/>
 </element>
@@
 <attribute name="VALUE" x="11.1807" y="23.9925" size="1.016" layer="28" ratio="12" rot="MR180"/>
 </element>
-<element name="JP1" library="pinhead" package="1X07" value="" x="4.5054" y="22.367375" smashed="yes" rot="R270">
+<element name="JP1" library="con-lsta" library_urn="urn:adsk.eagle:library:161" package="FE07" package3d_urn="urn:adsk.eagle:package:8223/1" override_package3d_urn="urn:adsk.eagle:package:48524428/2" override_package_urn="urn:adsk.eagle:footprint:8137/1" value="" x="4.5054" y="22.367375" smashed="yes" rot="R270">
+<attribute name="MF" value="" x="4.5054" y="22.367375" size="1.778" layer="27" rot="R270" display="off"/>
+<attribute name="MPN" value="" x="4.5054" y="22.367375" size="1.778" layer="27" rot="R270" display="off"/>
 <attribute name="NAME" x="3.1268" y="11.48995" size="1.27" layer="25" ratio="10"/>
+<attribute name="OC_FARNELL" value="unknown" x="4.5054" y="22.367375" size="1.778" layer="27" rot="R270" display="off"/>
+<attribute name="OC_NEWARK" value="unknown" x="4.5054" y="22.367375" size="1.778" layer="27" rot="R270" display="off"/>
+<attribute name="POPULARITY" value="3" x="4.5054" y="22.367375" size="1.778" layer="27" rot="R270" display="off"/>
 <attribute name="VALUE" x="1.3304" y="31.257375" size="1.27" layer="27" rot="R270"/>
 </element>
@@
 </drawing>
 <compatibility>
+<note version="8.2" severity="warning">
+Since Version 8.2, EAGLE supports online libraries. The ids
+of those online libraries will not be understood (or retained)
+with this version.
+</note>
 <note version="8.3" severity="warning">
 Since Version 8.3, EAGLE supports Fusion synchronisation.
@@
 packages will not be understood (or retained) with this version.
 </note>
+<note version="9.4" severity="warning">
+Since Version 9.4, EAGLE supports the overriding of 3D packages
+in schematics and board files. Those overridden 3d packages
+will not be understood (or retained) with this version.
+</note>
 </compatibility>
